Commit message: update world setup
Signed-off-by: Jaeyoung Lee <jylee0121@gmail.com>

File: urdf/udacity_bot.xacro (robot description, xacro)
@@ -1,4 +1,14 @@
 <?xml version='1.0'?>
 <robot name="udacity_bot" xmlns:xacro="http://www.ros.org/wiki/xacro">
+  <xacro:include filename="$(find udacity_bot)/urdf/udacity_bot.gazebo" />
+  <material name="red">
+    <color rgba="1.0 0.0 0.0 1.0" />
+  </material>
+  <material name="green">
+    <color rgba="0.0 1.0 0.0 1.0" />
+  </material>
+  <material name="blue">
+    <color rgba="0.0 0.0 1.0 1.0" />
+  </material>
   <link name="robot_footprint"></link>
   <joint name="robot_footprint_joint" type="fixed">
@@ -29,4 +39,5 @@
         <box size=".4 .2 .1"/>
       </geometry>
+      <material name="blue" />
     </visual>
     <collision name='back_caster_collision'>
@@ -86,4 +97,5 @@
         <cylinder radius="0.1" length="0.05" />
       </geometry>
+      <material name="green" />
     </visual>
   </link>
@@ -119,4 +131,5 @@
         <cylinder radius="0.1" length="0.05" />
       </geometry>
+      <material name="green" />
     </visual>
   </link>
@@ -149,4 +162,5 @@
         <box size="0.05 0.05 0.05" />
       </geometry>
+      <material name="red" />
     </visual>
   </link>
