Commit message: change the laser scanner setup: 180 degree to 360
Signed-off-by: Jaeyoung Lee <jylee0121@gmail.com>

File: urdf/my_bot.xacro (robot description, xacro)
@@ -29,15 +29,15 @@
     </inertial>
     <collision name='collision'>
-      <origin xyz="0 0 0" rpy=" 0 0 0"/>
+      <origin xyz="0 0 0.025" rpy=" 0 0 0"/>
       <geometry>
-        <box size=".4 .2 .1"/>
+        <box size=".4 .2 .15"/>
       </geometry>
     </collision>
     <visual name='chassis_visual'>
-      <origin xyz="0 0 0" rpy=" 0 0 0"/>
+      <origin xyz="0 0 0.025" rpy=" 0 0 0"/>
       <geometry>
-        <box size=".4 .2 .1"/>
+        <box size=".4 .2 .15"/>
       </geometry>
-      <material name="blue" />
+      <material name="red" />
     </visual>
     <collision name='back_caster_collision'>
@@ -167,5 +167,5 @@
   <!-- LASER RANGEFINDER -->
   <joint name="hokuyo_joint" type="fixed">
-    <origin xyz="0.15 0 0.1" rpy="0 0 0" />
+    <origin xyz="0.15 0 0.125" rpy="0 0 0" />
     <parent link="chassis" />
     <child link="hokuyo" />
